Commit message: 自动建图探索

File: src/my_robot_description/urdf/my_robot.urdf (robot description, URDF)
Before this commit: robot my_awesome_robot, 6 links, 5 joints
Links:
- link base_link: geometry collision cylinder length=0.12 radius=0.175; visual cylinder length=0.12 radius=0.175
- link imu_link: geometry collision box size=0.08 0.05 0.03; visual box size=0.08 0.05 0.03

Commit message: Milestone: validated navigation base and semantic mapping plan

File: src/my_robot_description/urdf/my_robot.urdf (robot description, URDF)
Before this commit: robot my_awesome_robot, 6 links, 5 joints
Joints:
- joint camera_color_screw_joint: origin xyz=0.1434 -0.0002 0.13933 rpy=3.1416 0 -0.0467 -> xyz=0.146327 -0.002217 0.342200 rpy=3.138477 -0.004836 -0.043870
